File: tests/simple.kicad_pcb (KiCad board)
At the start: 2 copper layers, 2 parts, among them U1 74AHC273, U2 74AHC273

Commit message: Fiddling with COG
Other:
- board outline added: 128.8 x 55.1 mm
